File: IOT_Hardware/EC-TDS-PPM/EC-TDS-PPM1_6.brd (EAGLE design)
At the start: 107.1 x 53.4 mm, 154 parts, among them IC1 TL084P, IC2 TL084P, IC3 TL084P, IC4 LINEAR_MC33269ST-3.3T3, J1 DCJ0202, J2 DCJ0202, J3 DCJ0202, Q1 VSK_N_FET_TO23, Q2 VSK_N_FET_TO23, Q3 VSK_N_FET_TO23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

Commit message: Arduino Project Bang Nguyen
Signed-off-by: BangNguyen <ndbn200491@gmail.com>
Routing:
- net GND1: vias 160 -> 161
Changed lines of the file:
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@@
 <via x="94.615" y="35.56" extent="1-16" drill="0.6096"/>
 <via x="95.758" y="35.56" extent="1-16" drill="0.6096"/>
+<via x="88.9" y="46.482" extent="1-16" drill="0.6096"/>
 </signal>
 <signal name="N$3">
@@
 <wire x1="104.14" y1="50.292" x2="104.14" y2="49.784" width="0.254" layer="16"/>
 <wire x1="104.14" y1="49.784" x2="104.394" y2="49.53" width="0.254" layer="16"/>
-<wire x1="97.409" y1="40.425" x2="97.409" y2="40.513" width="0" layer="19" extent="1-1"/>
+<wire x1="97.409" y1="40.513" x2="97.409" y2="40.425" width="0.254" layer="1"/>
 </signal>
 </signals>
