File: IOT_Hardware/EC-TDS-PPM/EC-TDS-PPM1_7.brd (EAGLE design)
At the start: 107.1 x 53.4 mm, 158 parts, among them IC1 TL084P, IC2 TL084P, IC3 TL084P, IC4 LINEAR_MC33269ST-3.3T3, J1 DCJ0202, J2 DCJ0202, J3 DCJ0202, Q1 VSK_N_FET_TO23, Q2 VSK_N_FET_TO23, Q3 VSK_N_FET_TO23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

Commit message: Bang Nguyen Completely First Demo
Signed-off-by: BangNguyen <ndbn200491@gmail.com>
Routing:
- net GND1: track 30.7 -> 29.3 mm
Changed lines of the file:
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@@
 <layer number="19" name="Unrouted" color="6" fill="1" visible="yes" active="yes"/>
 <layer number="20" name="Dimension" color="15" fill="1" visible="yes" active="yes"/>
-<layer number="21" name="tPlace" color="7" fill="1" visible="yes" active="yes"/>
-<layer number="22" name="bPlace" color="7" fill="1" visible="yes" active="yes"/>
+<layer number="21" name="tPlace" color="7" fill="1" visible="no" active="yes"/>
+<layer number="22" name="bPlace" color="7" fill="1" visible="no" active="yes"/>
 <layer number="23" name="tOrigins" color="15" fill="1" visible="yes" active="yes"/>
 <layer number="24" name="bOrigins" color="15" fill="1" visible="yes" active="yes"/>
@@
 <layer number="37" name="tTest" color="7" fill="1" visible="no" active="yes"/>
 <layer number="38" name="bTest" color="7" fill="1" visible="no" active="yes"/>
-<layer number="39" name="tKeepout" color="4" fill="11" visible="yes" active="yes"/>
+<layer number="39" name="tKeepout" color="4" fill="11" visible="no" active="yes"/>
 <layer number="40" name="bKeepout" color="1" fill="11" visible="no" active="yes"/>
-<layer number="41" name="tRestrict" color="4" fill="10" visible="yes" active="yes"/>
+<layer number="41" name="tRestrict" color="4" fill="10" visible="no" active="yes"/>
 <layer number="42" name="bRestrict" color="1" fill="10" visible="no" active="yes"/>
 <layer number="43" name="vRestrict" color="2" fill="10" visible="no" active="yes"/>
 <layer number="44" name="Drills" color="7" fill="1" visible="no" active="yes"/>
-<layer number="45" name="Holes" color="7" fill="1" visible="yes" active="yes"/>
+<layer number="45" name="Holes" color="7" fill="1" visible="no" active="yes"/>
 <layer number="46" name="Milling" color="3" fill="1" visible="no" active="yes"/>
 <layer number="47" name="Measures" color="7" fill="1" visible="no" active="yes"/>
@@
 <wire x1="87.249" y1="43.434" x2="88.9" y2="43.434" width="0.381" layer="1"/>
 <via x="88.9" y="43.434" extent="1-16" drill="0.6096"/>
-<wire x1="88.9" y1="43.434" x2="86.741" y2="43.307" width="0.381" layer="16"/>
-<wire x1="86.741" y1="43.307" x2="86.614" y2="43.434" width="0.381" layer="16"/>
+<wire x1="88.9" y1="43.434" x2="88.138" y2="43.307" width="0.381" layer="16"/>
+<wire x1="88.138" y1="43.307" x2="88.138" y2="43.18" width="0.381" layer="16"/>
 <via x="89.027" y="45.466" extent="1-16" drill="0.6096"/>
 <wire x1="89.154" y1="46.482" x2="89.154" y2="45.593" width="0.381" layer="1"/>
