File: IOT_Hardware/EC-TDS-PPM/EC-TDS-PPM_V2-1.brd (EAGLE design)
At the start: 107.1 x 60.6 mm, 123 parts, among them IC1 TL084D, IC2 TL082P, IC3 TL084P, IC4 LINEAR_MC33269ST-3.3T3, IC5 TL082D, Q1 NPN, Q7 32.768, X1 BU-SMA-H

Commit message: Bang Nguyen Signed-off-by: BangNguyen <ndbn200491@gmail.com>
Routing:
- net N$7: track 36.2 -> 38.8 mm
- net N$21: track 24.4 -> 25.1 mm
- net N$37: track 11.8 -> 12.4 mm
